Commit message: Refactor folder structure to follow ros conventions
Signed-off-by: Baoan Du <baoan.du.xj@renesas.com>

File: urdf/inspire_hand_left_macro.xacro (robot description, xacro)
@@ -27,5 +27,5 @@
         <origin xyz="0 0 0" rpy="0 0 0"/>
         <geometry>
-          <mesh filename="package://inspire_rh56_hand_description/urdf/meshes/visual/left_base_link.glb"/>
+          <mesh filename="package://inspire_rh56_hand_description/meshes/visual/left_base_link.glb"/>
         </geometry>
       </visual>
@@ -89,11 +89,11 @@
         <origin xyz="0 0 0" rpy="0 0 0"/>
         <geometry>
-          <mesh filename="package://inspire_rh56_hand_description/urdf/meshes/visual/left_thumb_proximal_base.glb"/>
-        </geometry>
-      </visual>
-      <collision>
-        <origin xyz="0 0 0" rpy="0 0 0"/>
-        <geometry>
-          <mesh filename="package://inspire_rh56_hand_description/urdf/meshes/collision/left_thumb_proximal_base.obj"/>
+          <mesh filename="package://inspire_rh56_hand_description/meshes/visual/left_thumb_proximal_base.glb"/>
+        </geometry>
+      </visual>
+      <collision>
+        <origin xyz="0 0 0" rpy="0 0 0"/>
+        <geometry>
+          <mesh filename="package://inspire_rh56_hand_description/meshes/collision/left_thumb_proximal_base.obj"/>
         </geometry>
       </collision>
@@ -116,11 +116,11 @@
         <origin xyz="0 0 0" rpy="0 0 0"/>
         <geometry>
-          <mesh filename="package://inspire_rh56_hand_description/urdf/meshes/visual/left_thumb_proximal.glb"/>
-        </geometry>
-      </visual>
-      <collision>
-        <origin xyz="0 0 0" rpy="0 0 0"/>
-        <geometry>
-          <mesh filename="package://inspire_rh56_hand_description/urdf/meshes/collision/left_thumb_proximal.obj"/>
+          <mesh filename="package://inspire_rh56_hand_description/meshes/visual/left_thumb_proximal.glb"/>
+        </geometry>
+      </visual>
+      <collision>
+        <origin xyz="0 0 0" rpy="0 0 0"/>
+        <geometry>
+          <mesh filename="package://inspire_rh56_hand_description/meshes/collision/left_thumb_proximal.obj"/>
         </geometry>
       </collision>
@@ -143,11 +143,11 @@
         <origin xyz="0 0 0" rpy="0 0 0"/>
         <geometry>
-          <mesh filename="package://inspire_rh56_hand_description/urdf/meshes/visual/left_thumb_intermediate.glb"/>
-        </geometry>
-      </visual>
-      <collision>
-        <origin xyz="0 0 0" rpy="0 0 0"/>
-        <geometry>
-          <mesh filename="package://inspire_rh56_hand_description/urdf/meshes/collision/left_thumb_intermediate.obj"/>
+          <mesh filename="package://inspire_rh56_hand_description/meshes/visual/left_thumb_intermediate.glb"/>
+        </geometry>
+      </visual>
+      <collision>
+        <origin xyz="0 0 0" rpy="0 0 0"/>
+        <geometry>
+          <mesh filename="package://inspire_rh56_hand_description/meshes/collision/left_thumb_intermediate.obj"/>
         </geometry>
       </collision>
@@ -171,11 +171,11 @@
         <origin xyz="0 0 0" rpy="0 0 0"/>
         <geometry>
-          <mesh filename="package://inspire_rh56_hand_description/urdf/meshes/visual/left_thumb_distal.glb"/>
-        </geometry>
-      </visual>
-      <collision>
-        <origin xyz="0 0 0" rpy="0 0 0"/>
-        <geometry>
-          <mesh filename="package://inspire_rh56_hand_description/urdf/meshes/collision/left_thumb_distal.obj"/>
+          <mesh filename="package://inspire_rh56_hand_description/meshes/visual/left_thumb_distal.glb"/>
+        </geometry>
+      </visual>
+      <collision>
+        <origin xyz="0 0 0" rpy="0 0 0"/>
+        <geometry>
+          <mesh filename="package://inspire_rh56_hand_description/meshes/collision/left_thumb_distal.obj"/>
         </geometry>
       </collision>
@@ -199,11 +199,11 @@
         <origin xyz="0 0 0" rpy="0 0 0"/>
         <geometry>
-          <mesh filename="package://inspire_rh56_hand_description/urdf/meshes/visual/left_index_proximal.glb"/>
-        </geometry>
-      </visual>
-      <collision>
-        <origin xyz="0 0 0" rpy="0 0 0"/>
-        <geometry>
-          <mesh filename="package://inspire_rh56_hand_description/urdf/meshes/collision/left_index_proximal.obj"/>
+          <mesh filename="package://inspire_rh56_hand_description/meshes/visual/left_index_proximal.glb"/>
+        </geometry>
+      </visual>
+      <collision>
+        <origin xyz="0 0 0" rpy="0 0 0"/>
+        <geometry>
+          <mesh filename="package://inspire_rh56_hand_description/meshes/collision/left_index_proximal.obj"/>
         </geometry>
       </collision>
@@ -226,11 +226,11 @@
         <origin xyz="0 0 0" rpy="0 0 0"/>
         <geometry>
-          <mesh filename="package://inspire_rh56_hand_description/urdf/meshes/visual/left_index_intermediate.glb"/>
-        </geometry>
-      </visual>
-      <collision>
-        <origin xyz="0 0 0" rpy="0 0 0"/>
-        <geometry>
-          <mesh filename="package://inspire_rh56_hand_description/urdf/meshes/collision/left_index_intermediate.obj"/>
+          <mesh filename="package://inspire_rh56_hand_description/meshes/visual/left_index_intermediate.glb"/>
+        </geometry>
+      </visual>
+      <collision>
+        <origin xyz="0 0 0" rpy="0 0 0"/>
+        <geometry>
+          <mesh filename="package://inspire_rh56_hand_description/meshes/collision/left_index_intermediate.obj"/>
         </geometry>
       </collision>
@@ -254,11 +254,11 @@
         <origin xyz="0 0 0" rpy="0 0 0"/>
         <geometry>
-          <mesh filename="package://inspire_rh56_hand_description/urdf/meshes/visual/left_index_proximal.glb"/>
-        </geometry>
-      </visual>
-      <collision>
-        <origin xyz="0 0 0" rpy="0 0 0"/>
-        <geometry>
-          <mesh filename="package://inspire_rh56_hand_description/urdf/meshes/collision/left_index_proximal.obj"/>
+          <mesh filename="package://inspire_rh56_hand_description/meshes/visual/left_index_proximal.glb"/>
+        </geometry>
+      </visual>
+      <collision>
+        <origin xyz="0 0 0" rpy="0 0 0"/>
+        <geometry>
+          <mesh filename="package://inspire_rh56_hand_description/meshes/collision/left_index_proximal.obj"/>
         </geometry>
       </collision>
@@ -281,11 +281,11 @@
         <origin xyz="0 0 0" rpy="0 0 0"/>
         <geometry>
-          <mesh filename="package://inspire_rh56_hand_description/urdf/meshes/visual/left_middle_intermediate.glb"/>
-        </geometry>
-      </visual>
-      <collision>
-        <origin xyz="0 0 0" rpy="0 0 0"/>
-        <geometry>
-          <mesh filename="package://inspire_rh56_hand_description/urdf/meshes/collision/left_middle_intermediate.obj"/>
+          <mesh filename="package://inspire_rh56_hand_description/meshes/visual/left_middle_intermediate.glb"/>
+        </geometry>
+      </visual>
+      <collision>
+        <origin xyz="0 0 0" rpy="0 0 0"/>
+        <geometry>
+          <mesh filename="package://inspire_rh56_hand_description/meshes/collision/left_middle_intermediate.obj"/>
         </geometry>
       </collision>
@@ -309,11 +309,11 @@
         <origin xyz="0 0 0" rpy="0 0 0"/>
         <geometry>
-          <mesh filename="package://inspire_rh56_hand_description/urdf/meshes/visual/left_index_proximal.glb"/>
-        </geometry>
-      </visual>
-      <collision>
-        <origin xyz="0 0 0" rpy="0 0 0"/>
-        <geometry>
-          <mesh filename="package://inspire_rh56_hand_description/urdf/meshes/collision/left_index_proximal.obj"/>
+          <mesh filename="package://inspire_rh56_hand_description/meshes/visual/left_index_proximal.glb"/>
+        </geometry>
+      </visual>
+      <collision>
+        <origin xyz="0 0 0" rpy="0 0 0"/>
+        <geometry>
+          <mesh filename="package://inspire_rh56_hand_description/meshes/collision/left_index_proximal.obj"/>
         </geometry>
       </collision>
@@ -336,11 +336,11 @@
         <origin xyz="0 0 0" rpy="0 0 0"/>
         <geometry>
-          <mesh filename="package://inspire_rh56_hand_description/urdf/meshes/visual/left_index_intermediate.glb"/>
-        </geometry>
-      </visual>
-      <collision>
-        <origin xyz="0 0 0" rpy="0 0 0"/>
-        <geometry>
-          <mesh filename="package://inspire_rh56_hand_description/urdf/meshes/collision/left_index_intermediate.obj"/>
+          <mesh filename="package://inspire_rh56_hand_description/meshes/visual/left_index_intermediate.glb"/>
+        </geometry>
+      </visual>
+      <collision>
+        <origin xyz="0 0 0" rpy="0 0 0"/>
+        <geometry>
+          <mesh filename="package://inspire_rh56_hand_description/meshes/collision/left_index_intermediate.obj"/>
         </geometry>
       </collision>
@@ -364,11 +364,11 @@
         <origin xyz="0 0 0" rpy="0 0 0"/>
         <geometry>
-          <mesh filename="package://inspire_rh56_hand_description/urdf/meshes/visual/left_index_proximal.glb"/>
-        </geometry>
-      </visual>
-      <collision>
-        <origin xyz="0 0 0" rpy="0 0 0"/>
-        <geometry>
-          <mesh filename="package://inspire_rh56_hand_description/urdf/meshes/collision/left_index_proximal.obj"/>
+          <mesh filename="package://inspire_rh56_hand_description/meshes/visual/left_index_proximal.glb"/>
+        </geometry>
+      </visual>
+      <collision>
+        <origin xyz="0 0 0" rpy="0 0 0"/>
+        <geometry>
+          <mesh filename="package://inspire_rh56_hand_description/meshes/collision/left_index_proximal.obj"/>
         </geometry>
       </collision>
@@ -391,11 +391,11 @@
         <origin xyz="0 0 0" rpy="0 0 0"/>
         <geometry>
-          <mesh filename="package://inspire_rh56_hand_description/urdf/meshes/visual/left_pinky_intermediate.glb"/>
-        </geometry>
-      </visual>
-      <collision>
-        <origin xyz="0 0 0" rpy="0 0 0"/>
-        <geometry>
-          <mesh filename="package://inspire_rh56_hand_description/urdf/meshes/collision/left_pinky_intermediate.obj"/>
+          <mesh filename="package://inspire_rh56_hand_description/meshes/visual/left_pinky_intermediate.glb"/>
+        </geometry>
+      </visual>
+      <collision>
+        <origin xyz="0 0 0" rpy="0 0 0"/>
+        <geometry>
+          <mesh filename="package://inspire_rh56_hand_description/meshes/collision/left_pinky_intermediate.obj"/>
         </geometry>
       </collision>

File: urdf/inspire_hand_right_macro.xacro (robot description, xacro)
@@ -27,5 +27,5 @@
         <origin xyz="0 0 0" rpy="0 0 0"/>
         <geometry>
-          <mesh filename="package://inspire_rh56_hand_description/urdf/meshes/visual/right_base_link.glb"/>
+          <mesh filename="package://inspire_rh56_hand_description/meshes/visual/right_base_link.glb"/>
         </geometry>
       </visual>
@@ -89,11 +89,11 @@
         <origin xyz="0 0 0" rpy="0 0 0"/>
         <geometry>
-          <mesh filename="package://inspire_rh56_hand_description/urdf/meshes/visual/right_thumb_proximal_base.glb"/>
-        </geometry>
-      </visual>
-      <collision>
-        <origin xyz="0 0 0" rpy="0 0 0"/>
-        <geometry>
-          <mesh filename="package://inspire_rh56_hand_description/urdf/meshes/collision/right_thumb_proximal_base.obj"/>
+          <mesh filename="package://inspire_rh56_hand_description/meshes/visual/right_thumb_proximal_base.glb"/>
+        </geometry>
+      </visual>
+      <collision>
+        <origin xyz="0 0 0" rpy="0 0 0"/>
+        <geometry>
+          <mesh filename="package://inspire_rh56_hand_description/meshes/collision/right_thumb_proximal_base.obj"/>
         </geometry>
       </collision>
@@ -116,11 +116,11 @@
         <origin xyz="0 0 0" rpy="0 0 0"/>
         <geometry>
-          <mesh filename="package://inspire_rh56_hand_description/urdf/meshes/visual/right_thumb_proximal.glb"/>
-        </geometry>
-      </visual>
-      <collision>
-        <origin xyz="0 0 0" rpy="0 0 0"/>
-        <geometry>
-          <mesh filename="package://inspire_rh56_hand_description/urdf/meshes/collision/right_thumb_proximal.obj"/>
+          <mesh filename="package://inspire_rh56_hand_description/meshes/visual/right_thumb_proximal.glb"/>
+        </geometry>
+      </visual>
+      <collision>
+        <origin xyz="0 0 0" rpy="0 0 0"/>
+        <geometry>
+          <mesh filename="package://inspire_rh56_hand_description/meshes/collision/right_thumb_proximal.obj"/>
         </geometry>
       </collision>
@@ -143,11 +143,11 @@
         <origin xyz="0 0 0" rpy="0 0 0"/>
         <geometry>
-          <mesh filename="package://inspire_rh56_hand_description/urdf/meshes/visual/right_thumb_intermediate.glb"/>
-        </geometry>
-      </visual>
-      <collision>
-        <origin xyz="0 0 0" rpy="0 0 0"/>
-        <geometry>
-          <mesh filename="package://inspire_rh56_hand_description/urdf/meshes/collision/right_thumb_intermediate.obj"/>
+          <mesh filename="package://inspire_rh56_hand_description/meshes/visual/right_thumb_intermediate.glb"/>
+        </geometry>
+      </visual>
+      <collision>
+        <origin xyz="0 0 0" rpy="0 0 0"/>
+        <geometry>
+          <mesh filename="package://inspire_rh56_hand_description/meshes/collision/right_thumb_intermediate.obj"/>
         </geometry>
       </collision>
@@ -171,11 +171,11 @@
         <origin xyz="0 0 0" rpy="0 0 0"/>
         <geometry>
-          <mesh filename="package://inspire_rh56_hand_description/urdf/meshes/visual/right_thumb_distal.glb"/>
-        </geometry>
-      </visual>
-      <collision>
-        <origin xyz="0 0 0" rpy="0 0 0"/>
-        <geometry>
-          <mesh filename="package://inspire_rh56_hand_description/urdf/meshes/collision/right_thumb_distal.obj"/>
+          <mesh filename="package://inspire_rh56_hand_description/meshes/visual/right_thumb_distal.glb"/>
+        </geometry>
+      </visual>
+      <collision>
+        <origin xyz="0 0 0" rpy="0 0 0"/>
+        <geometry>
+          <mesh filename="package://inspire_rh56_hand_description/meshes/collision/right_thumb_distal.obj"/>
         </geometry>
       </collision>
@@ -199,11 +199,11 @@
         <origin xyz="0 0 0" rpy="0 0 0"/>
         <geometry>
-          <mesh filename="package://inspire_rh56_hand_description/urdf/meshes/visual/right_index_proximal.glb"/>
-        </geometry>
-      </visual>
-      <collision>
-        <origin xyz="0 0 0" rpy="0 0 0"/>
-        <geometry>
-          <mesh filename="package://inspire_rh56_hand_description/urdf/meshes/collision/right_index_proximal.obj"/>
+          <mesh filename="package://inspire_rh56_hand_description/meshes/visual/right_index_proximal.glb"/>
+        </geometry>
+      </visual>
+      <collision>
+        <origin xyz="0 0 0" rpy="0 0 0"/>
+        <geometry>
+          <mesh filename="package://inspire_rh56_hand_description/meshes/collision/right_index_proximal.obj"/>
         </geometry>
       </collision>
@@ -226,11 +226,11 @@
         <origin xyz="0 0 0" rpy="0 0 0"/>
         <geometry>
-          <mesh filename="package://inspire_rh56_hand_description/urdf/meshes/visual/right_index_intermediate.glb"/>
-        </geometry>
-      </visual>
-      <collision>
-        <origin xyz="0 0 0" rpy="0 0 0"/>
-        <geometry>
-          <mesh filename="package://inspire_rh56_hand_description/urdf/meshes/collision/right_index_intermediate.obj"/>
+          <mesh filename="package://inspire_rh56_hand_description/meshes/visual/right_index_intermediate.glb"/>
+        </geometry>
+      </visual>
+      <collision>
+        <origin xyz="0 0 0" rpy="0 0 0"/>
+        <geometry>
+          <mesh filename="package://inspire_rh56_hand_description/meshes/collision/right_index_intermediate.obj"/>
         </geometry>
       </collision>
@@ -254,11 +254,11 @@
         <origin xyz="0 0 0" rpy="0 0 0"/>
         <geometry>
-          <mesh filename="package://inspire_rh56_hand_description/urdf/meshes/visual/right_index_proximal.glb"/>
-        </geometry>
-      </visual>
-      <collision>
-        <origin xyz="0 0 0" rpy="0 0 0"/>
-        <geometry>
-          <mesh filename="package://inspire_rh56_hand_description/urdf/meshes/collision/right_index_proximal.obj"/>
+          <mesh filename="package://inspire_rh56_hand_description/meshes/visual/right_index_proximal.glb"/>
+        </geometry>
+      </visual>
+      <collision>
+        <origin xyz="0 0 0" rpy="0 0 0"/>
+        <geometry>
+          <mesh filename="package://inspire_rh56_hand_description/meshes/collision/right_index_proximal.obj"/>
         </geometry>
       </collision>
@@ -281,11 +281,11 @@
         <origin xyz="0 0 0" rpy="0 0 0"/>
         <geometry>
-          <mesh filename="package://inspire_rh56_hand_description/urdf/meshes/visual/right_middle_intermediate.glb"/>
-        </geometry>
-      </visual>
-      <collision>
-        <origin xyz="0 0 0" rpy="0 0 0"/>
-        <geometry>
-          <mesh filename="package://inspire_rh56_hand_description/urdf/meshes/collision/right_middle_intermediate.obj"/>
+          <mesh filename="package://inspire_rh56_hand_description/meshes/visual/right_middle_intermediate.glb"/>
+        </geometry>
+      </visual>
+      <collision>
+        <origin xyz="0 0 0" rpy="0 0 0"/>
+        <geometry>
+          <mesh filename="package://inspire_rh56_hand_description/meshes/collision/right_middle_intermediate.obj"/>
         </geometry>
       </collision>
@@ -309,11 +309,11 @@
         <origin xyz="0 0 0" rpy="0 0 0"/>
         <geometry>
-          <mesh filename="package://inspire_rh56_hand_description/urdf/meshes/visual/right_index_proximal.glb"/>
-        </geometry>
-      </visual>
-      <collision>
-        <origin xyz="0 0 0" rpy="0 0 0"/>
-        <geometry>
-          <mesh filename="package://inspire_rh56_hand_description/urdf/meshes/collision/right_index_proximal.obj"/>
+          <mesh filename="package://inspire_rh56_hand_description/meshes/visual/right_index_proximal.glb"/>
+        </geometry>
+      </visual>
+      <collision>
+        <origin xyz="0 0 0" rpy="0 0 0"/>
+        <geometry>
+          <mesh filename="package://inspire_rh56_hand_description/meshes/collision/right_index_proximal.obj"/>
         </geometry>
       </collision>
@@ -336,11 +336,11 @@
         <origin xyz="0 0 0" rpy="0 0 0"/>
         <geometry>
-          <mesh filename="package://inspire_rh56_hand_description/urdf/meshes/visual/right_index_intermediate.glb"/>
-        </geometry>
-      </visual>
-      <collision>
-        <origin xyz="0 0 0" rpy="0 0 0"/>
-        <geometry>
-          <mesh filename="package://inspire_rh56_hand_description/urdf/meshes/collision/right_index_intermediate.obj"/>
+          <mesh filename="package://inspire_rh56_hand_description/meshes/visual/right_index_intermediate.glb"/>
+        </geometry>
+      </visual>
+      <collision>
+        <origin xyz="0 0 0" rpy="0 0 0"/>
+        <geometry>
+          <mesh filename="package://inspire_rh56_hand_description/meshes/collision/right_index_intermediate.obj"/>
         </geometry>
       </collision>
@@ -364,11 +364,11 @@
         <origin xyz="0 0 0" rpy="0 0 0"/>
         <geometry>
-          <mesh filename="package://inspire_rh56_hand_description/urdf/meshes/visual/right_index_proximal.glb"/>
-        </geometry>
-      </visual>
-      <collision>
-        <origin xyz="0 0 0" rpy="0 0 0"/>
-        <geometry>
-          <mesh filename="package://inspire_rh56_hand_description/urdf/meshes/collision/right_index_proximal.obj"/>
+          <mesh filename="package://inspire_rh56_hand_description/meshes/visual/right_index_proximal.glb"/>
+        </geometry>
+      </visual>
+      <collision>
+        <origin xyz="0 0 0" rpy="0 0 0"/>
+        <geometry>
+          <mesh filename="package://inspire_rh56_hand_description/meshes/collision/right_index_proximal.obj"/>
         </geometry>
       </collision>
@@ -391,11 +391,11 @@
         <origin xyz="0 0 0" rpy="0 0 0"/>
         <geometry>
-          <mesh filename="package://inspire_rh56_hand_description/urdf/meshes/visual/right_pinky_intermediate.glb"/>
-        </geometry>
-      </visual>
-      <collision>
-        <origin xyz="0 0 0" rpy="0 0 0"/>
-        <geometry>
-          <mesh filename="package://inspire_rh56_hand_description/urdf/meshes/collision/right_pinky_intermediate.obj"/>
+          <mesh filename="package://inspire_rh56_hand_description/meshes/visual/right_pinky_intermediate.glb"/>
+        </geometry>
+      </visual>
+      <collision>
+        <origin xyz="0 0 0" rpy="0 0 0"/>
+        <geometry>
+          <mesh filename="package://inspire_rh56_hand_description/meshes/collision/right_pinky_intermediate.obj"/>
         </geometry>
       </collision>
