Commit message: Refactor folder structure to follow ros conventions
Signed-off-by: Baoan Du <baoan.du.xj@renesas.com>

File: urdf/reference/inspire_hand_left_ref.urdf (robot description, URDF)
Before this commit: robot inspire_hand_left, 20 links, 19 joints
Links:
- link hand_base_link: geometry collision box size=0.0125 0.0111 0.0089; collision box size=0.0125 0.0111 0.0089
- link index_intermediate: geometry collision mesh filename=package://inspire_rh56_urdf/meshes/collision/left_index_int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; visual mesh filename=package://inspire_rh56_urdf/meshes/visual/left_index_interm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
- link index_proximal: geometry collision mesh filename=package://inspire_rh56_urdf/meshes/collision/left_index_pro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; visual mesh filename=package://inspire_rh56_urdf/meshes/visual/left_index_proxim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
- link middle_intermediate: geometry collision mesh filename=package://inspire_rh56_urdf/meshes/collision/left_middle_in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; visual mesh filename=package://inspire_rh56_urdf/meshes/visual/left_middle_inter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
- link middle_proximal: geometry collision mesh filename=package://inspire_rh56_urdf/meshes/collision/left_index_pro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; visual mesh filename=package://inspire_rh56_urdf/meshes/visual/left_index_proxim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
- link pinky_intermediate: geometry collision mesh filename=package://inspire_rh56_urdf/meshes/collision/left_pinky_int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; visual mesh filename=package://inspire_rh56_urdf/meshes/visual/left_pinky_interm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
- link pinky_proximal: geometry collision mesh filename=package://inspire_rh56_urdf/meshes/collision/left_index_pro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; visual mesh filename=package://inspire_rh56_urdf/meshes/visual/left_index_proxim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
- link ring_intermediate: geometry collision mesh filename=package://inspire_rh56_urdf/meshes/collision/left_index_int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; visual mesh filename=package://inspire_rh56_urdf/meshes/visual/left_index_interm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
- link ring_proximal: geometry collision mesh filename=package://inspire_rh56_urdf/meshes/collision/left_index_pro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; visual mesh filename=package://inspire_rh56_urdf/meshes/visual/left_index_proxim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
- link thumb_distal: geometry collision mesh filename=package://inspire_rh56_urdf/meshes/collision/left_thumb_dis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 scale=1 1 1; visual mesh filename=package://inspire_rh56_urdf/meshes/visual/left_thumb_distal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
- link thumb_intermediate: geometry collision mesh filename=package://inspire_rh56_urdf/meshes/collision/left_thumb_int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; visual mesh filename=package://inspire_rh56_urdf/meshes/visual/left_thumb_interm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
- link thumb_proximal: geometry collision mesh filename=package://inspire_rh56_urdf/meshes/collision/left_thumb_pro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; visual mesh filename=package://inspire_rh56_urdf/meshes/visual/left_thumb_proxim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
- link thumb_proximal_base: geometry collision mesh filename=package://inspire_rh56_urdf/meshes/collision/left_thumb_pro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; visual mesh filename=package://inspire_rh56_urdf/meshes/visual/left_thumb_proxim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

File: urdf/reference/inspire_hand_right_ref.urdf (robot description, URDF)
Before this commit: robot inspire_hand_right, 19 links, 18 joints
Links:
- link hand_base_link: geometry collision box size=0.0125 0.0111 0.0089; collision box size=0.0125 0.0111 0.0089
- link index_intermediate: geometry collision mesh filename=package://inspire_rh56_urdf/meshes/collision/right_index_in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; visual mesh filename=package://inspire_rh56_urdf/meshes/visual/right_index_inter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
- link index_proximal: geometry collision mesh filename=package://inspire_rh56_urdf/meshes/collision/right_index_pr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; visual mesh filename=package://inspire_rh56_urdf/meshes/visual/right_index_proxi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
- link middle_intermediate: geometry collision mesh filename=package://inspire_rh56_urdf/meshes/collision/right_middle_i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; visual mesh filename=package://inspire_rh56_urdf/meshes/visual/right_middle_inte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
- link middle_proximal: geometry collision mesh filename=package://inspire_rh56_urdf/meshes/collision/right_index_pr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; visual mesh filename=package://inspire_rh56_urdf/meshes/visual/right_index_proxi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
- link pinky_intermediate: geometry collision mesh filename=package://inspire_rh56_urdf/meshes/collision/right_pinky_in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; visual mesh filename=package://inspire_rh56_urdf/meshes/visual/right_pinky_inter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
- link pinky_proximal: geometry collision mesh filename=package://inspire_rh56_urdf/meshes/collision/right_index_pr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; visual mesh filename=package://inspire_rh56_urdf/meshes/visual/right_index_proxi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
- link ring_intermediate: geometry collision mesh filename=package://inspire_rh56_urdf/meshes/collision/right_index_in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; visual mesh filename=package://inspire_rh56_urdf/meshes/visual/right_index_inter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
- link ring_proximal: geometry collision mesh filename=package://inspire_rh56_urdf/meshes/collision/right_index_pr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; visual mesh filename=package://inspire_rh56_urdf/meshes/visual/right_index_proxi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
- link thumb_distal: geometry collision mesh filename=package://inspire_rh56_urdf/meshes/collision/right_thumb_di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; visual mesh filename=package://inspire_rh56_urdf/meshes/visual/right_thumb_dista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
- link thumb_intermediate: geometry collision mesh filename=package://inspire_rh56_urdf/meshes/collision/right_thumb_in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; visual mesh filename=package://inspire_rh56_urdf/meshes/visual/right_thumb_inter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
- link thumb_proximal: geometry collision mesh filename=package://inspire_rh56_urdf/meshes/collision/right_thumb_pr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; visual mesh filename=package://inspire_rh56_urdf/meshes/visual/right_thumb_proxi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
- link thumb_proximal_base: geometry collision mesh filename=package://inspire_rh56_urdf/meshes/collision/right_thumb_pr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; visual mesh filename=package://inspire_rh56_urdf/meshes/visual/right_thumb_proxi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

Commit message: Increase velocity limits for Inspire hand joints
Signed-off-by: Dat Nguyen <dat.nguyen.dn@bp.renesas.com>

File: urdf/inspire_hand_left_macro.xacro (robot description, xacro)
@@ -104,5 +104,5 @@
       <child link="${prefix}thumb_proximal_base"/>
       <axis xyz="0 0 1"/>
-      <limit lower="0" upper="1.308" effort="1" velocity="0.5"/>
+      <limit lower="0" upper="1.308" effort="1" velocity="1.635"/>
     </joint>
     <!-- Thumb proximal -->
@@ -131,5 +131,5 @@
       <child link="${prefix}thumb_proximal"/>
       <axis xyz="0 0 -1"/>
-      <limit lower="0" upper="0.6" effort="1" velocity="0.5"/>
+      <limit lower="0" upper="0.6" effort="1" velocity="0.75"/>
     </joint>
     <!-- Thumb intermediate -->
@@ -158,5 +158,5 @@
       <child link="${prefix}thumb_intermediate"/>
       <axis xyz="0 0 -1"/>
-      <limit lower="0" upper="0.8" effort="1" velocity="0.5"/>
+      <limit lower="0" upper="0.8" effort="1" velocity="1"/>
       <mimic joint="${prefix}thumb_proximal_pitch_joint" multiplier="1.334" offset="0"/>
     </joint>
@@ -214,5 +214,5 @@
       <child link="${prefix}index_proximal"/>
       <axis xyz="0 0 -1"/>
-      <limit lower="0" upper="1.47" effort="1" velocity="0.5"/>
+      <limit lower="0" upper="1.47" effort="1" velocity="1.8375"/>
     </joint>
     <!-- Index finger intermediate -->
@@ -241,5 +241,5 @@
       <child link="${prefix}index_intermediate"/>
       <axis xyz="0 0 -1"/>
-      <limit lower="-0.04545" upper="1.56" effort="1" velocity="0.5"/>
+      <limit lower="-0.04545" upper="1.56" effort="1" velocity="2.0068"/>
       <mimic joint="${prefix}index_proximal_joint" multiplier="1.06399" offset="-0.04545"/>
     </joint>
@@ -269,5 +269,5 @@
       <child link="${prefix}middle_proximal"/>
       <axis xyz="0 0 -1"/>
-      <limit lower="0" upper="1.47" effort="1" velocity="0.5"/>
+      <limit lower="0" upper="1.47" effort="1" velocity="1.8375"/>
     </joint>
     <!-- Middle finger intermediate -->
@@ -296,5 +296,5 @@
       <child link="${prefix}middle_intermediate"/>
       <axis xyz="0 0 -1"/>
-      <limit lower="-0.04545" upper="1.56" effort="1" velocity="0.5"/>
+      <limit lower="-0.04545" upper="1.56" effort="1" velocity="2.0068"/>
       <mimic joint="${prefix}middle_proximal_joint" multiplier="1.06399" offset="-0.04545"/>
     </joint>
@@ -324,5 +324,5 @@
       <child link="${prefix}ring_proximal"/>
       <axis xyz="0 0 -1"/>
-      <limit lower="0" upper="1.47" effort="1" velocity="0.5"/>
+      <limit lower="0" upper="1.47" effort="1" velocity="1.8375"/>
     </joint>
     <!-- Ring finger intermediate -->
@@ -351,5 +351,5 @@
       <child link="${prefix}ring_intermediate"/>
       <axis xyz="0 0 -1"/>
-      <limit lower="-0.04545" upper="1.56" effort="1" velocity="0.5"/>
+      <limit lower="-0.04545" upper="1.56" effort="1" velocity="2.0068"/>
       <mimic joint="${prefix}ring_proximal_joint" multiplier="1.06399" offset="-0.04545"/>
     </joint>
@@ -379,5 +379,5 @@
       <child link="${prefix}pinky_proximal"/>
       <axis xyz="0 0 -1"/>
-      <limit lower="0" upper="1.47" effort="1" velocity="0.5"/>
+      <limit lower="0" upper="1.47" effort="1" velocity="1.8375"/>
     </joint>
     <!-- Pinky finger intermediate -->
@@ -406,5 +406,5 @@
       <child link="${prefix}pinky_intermediate"/>
       <axis xyz="0 0 -1"/>
-      <limit lower="-0.04545" upper="1.56" effort="1" velocity="0.5"/>
+      <limit lower="-0.04545" upper="1.56" effort="1" velocity="2.0068"/>
       <mimic joint="${prefix}pinky_proximal_joint" multiplier="1.06399" offset="-0.04545"/>
     </joint>

File: urdf/inspire_hand_right_macro.xacro (robot description, xacro)
@@ -104,5 +104,5 @@
       <child link="${prefix}thumb_proximal_base"/>
       <axis xyz="0 0 -1"/>
-      <limit lower="0.0" upper="1.308" effort="1" velocity="0.5"/>
+      <limit lower="0.0" upper="1.308" effort="1" velocity="1.635"/>
     </joint>
     <!-- Thumb proximal -->
@@ -131,5 +131,5 @@
       <child link="${prefix}thumb_proximal"/>
       <axis xyz="0 0 1"/>
-      <limit lower="0" upper="0.6" effort="1" velocity="0.5"/>
+      <limit lower="0" upper="0.6" effort="1" velocity="0.75"/>
     </joint>
     <!-- Thumb intermediate -->
@@ -158,5 +158,5 @@
       <child link="${prefix}thumb_intermediate"/>
       <axis xyz="0 0 1"/>
-      <limit lower="0" upper="0.8" effort="1" velocity="0.5"/>
+      <limit lower="0" upper="0.8" effort="1" velocity="1.0"/>
       <mimic joint="${prefix}thumb_proximal_pitch_joint" multiplier="1.334" offset="0"/>
     </joint>
@@ -214,5 +214,5 @@
       <child link="${prefix}index_proximal"/>
       <axis xyz="0 0 1"/>
-      <limit lower="0" upper="1.47" effort="1" velocity="0.5"/>
+      <limit lower="0" upper="1.47" effort="1" velocity="1.8375"/>
     </joint>
     <!-- Index finger intermediate -->
@@ -241,5 +241,5 @@
       <child link="${prefix}index_intermediate"/>
       <axis xyz="0 0 1"/>
-      <limit lower="-0.04545" upper="1.56" effort="1" velocity="0.5"/>
+      <limit lower="-0.04545" upper="1.56" effort="1" velocity="2.0068"/>
       <mimic joint="${prefix}index_proximal_joint" multiplier="1.06399" offset="-0.04545"/>
     </joint>
@@ -269,5 +269,5 @@
       <child link="${prefix}middle_proximal"/>
       <axis xyz="0 0 1"/>
-      <limit lower="0" upper="1.47" effort="1" velocity="0.5"/>
+      <limit lower="0" upper="1.47" effort="1" velocity="1.8375"/>
     </joint>
     <!-- Middle finger intermediate -->
@@ -296,5 +296,5 @@
       <child link="${prefix}middle_intermediate"/>
       <axis xyz="0 0 1"/>
-      <limit lower="-0.04545" upper="1.56" effort="1" velocity="0.5"/>
+      <limit lower="-0.04545" upper="1.56" effort="1" velocity="2.0068"/>
       <mimic joint="${prefix}middle_proximal_joint" multiplier="1.06399" offset="-0.04545"/>
     </joint>
@@ -324,5 +324,5 @@
       <child link="${prefix}ring_proximal"/>
       <axis xyz="0 0 1"/>
-      <limit lower="0" upper="1.47" effort="1" velocity="0.5"/>
+      <limit lower="0" upper="1.47" effort="1" velocity="1.8375"/>
     </joint>
     <!-- Ring finger intermediate -->
@@ -351,5 +351,5 @@
       <child link="${prefix}ring_intermediate"/>
       <axis xyz="0 0 1"/>
-      <limit lower="-0.04545" upper="1.56" effort="1" velocity="0.5"/>
+      <limit lower="-0.04545" upper="1.56" effort="1" velocity="2.0068"/>
       <mimic joint="${prefix}ring_proximal_joint" multiplier="1.06399" offset="-0.04545"/>
     </joint>
@@ -379,5 +379,5 @@
       <child link="${prefix}pinky_proximal"/>
       <axis xyz="0 0 1"/>
-      <limit lower="0" upper="1.47" effort="1" velocity="0.5"/>
+      <limit lower="0" upper="1.47" effort="1" velocity="1.8375"/>
     </joint>
     <!-- Pinky finger intermediate -->
@@ -406,5 +406,5 @@
       <child link="${prefix}pinky_intermediate"/>
       <axis xyz="0 0 1"/>
-      <limit lower="-0.04545" upper="1.56" effort="1" velocity="0.5"/>
+      <limit lower="-0.04545" upper="1.56" effort="1" velocity="2.0068"/>
       <mimic joint="${prefix}pinky_proximal_joint" multiplier="1.06399" offset="-0.04545"/>
     </joint>
